File: SW6RL4/hardware/1.0/kicad/SW6RL4.kicad_pcb (KiCad board)
At the start: 2 copper layers, 75 x 75 mm, 49 parts, among them J1 ANALOG_A, J10 Screw_Terminal_01x02, J2 ANALOG_B, J3 SB1, J4 SB0, J5 SB1, J6 Screw_Terminal_01x02, J7 Screw_Terminal_01x02, J8 CAN, J9 Screw_Terminal_01x02, K1 FINDER-32.21-x300, K2 FINDER-32.21-x300, K3 FINDER-32.21-x300, K4 FINDER-32.21-x300, SW1 MODE_ADDRESS, U1 Teensy_3.2, U2 CNY74-2H, U3 CNY74-2H, U4 CNY74-2H, U5 ULN2803A, U6 MCP2551-I-P, U7 TMR-1-1211

Commit message: Big refactor for new board
Parts:
- added SW2: PUSH_1, Button_Switch_THT:SW_PUSH_6mm, F.Cu at (142.4, 155.7)
- added SW3: PUSH_2, Button_Switch_THT:SW_PUSH_6mm, F.Cu at (142.4, 141.7)
- U1: value Teensy_3.2 -> Teensy_3.2-PDJR; footprint PDJR:DIP-28_W15.24mm_Socket -> PDJR:Teensy_3.2
- U2: value CNY74-2H -> TMR-1-1211; footprint Package_DIP:DIP-8_W7.62mm -> PDJR:TMR-1-1211
- U7: value TMR-1-1211 -> CNY74-2H; footprint PDJR:TMR-1-1211 -> Package_DIP:DIP-8_W7.62mm
- moved U7 35.3 mm to (175.4, 120.1), turned to 180 degrees
- moved U2 33.1 mm to (207.7, 105.4), turned to 270 degrees
- moved U4 11.2 mm to (175.4, 109.0)
- moved U3 11.2 mm to (175.4, 97.8)
Connections:
- U1 pad 10: /SWITCH_5 -> /PUSH_1
- U1 pad 9: /SWITCH_6 -> /PUSH_2
- U2 pad 1: Net-(R1-Pad2) -> /NET_C
- U2 pad 2: Net-(D1-Pad2) -> Net-(F1-Pad2)
- U2 pad 4: Net-(R2-Pad2) -> +5V
- U2 pad 6: /SWITCH_1 -> GND
- U3 pad 1: Net-(R3-Pad2) -> Net-(R1-Pad2)
- U3 pad 2: Net-(D3-Pad2) -> Net-(D1-Pad2)
- U3 pad 3: Net-(D4-Pad2) -> Net-(D2-Pad2)
- U3 pad 4: Net-(R4-Pad2) -> Net-(R2-Pad2)
- U3 pad 6: /SWITCH_3 -> /SWITCH_1
- U3 pad 7: /SWITCH_4 -> /SWITCH_2
- U4 pad 1: Net-(R5-Pad2) -> Net-(R3-Pad2)
- U4 pad 2: Net-(D5-Pad2) -> Net-(D3-Pad2)
- U4 pad 3: Net-(D6-Pad2) -> Net-(D4-Pad2)
- U4 pad 4: Net-(R6-Pad2) -> Net-(R4-Pad2)
- U4 pad 6: /SWITCH_5 -> /SWITCH_3
- U4 pad 7: /SWITCH_6 -> /SWITCH_4
- U7 pad 1: Net-(F1-Pad2) -> Net-(R5-Pad2)
- U7 pad 2: /NET_C -> Net-(D5-Pad2)
- U7 pad 4: GND -> Net-(R6-Pad2)
- U7 pad 6: +5V -> /PUSH_1
Routing:
- net /PUSH_1: track 0.00 -> 130.7 mm
- net /PUSH_2: track 0.00 -> 117.8 mm
- net /SWITCH_6: track 16.0 -> 0.00 mm
- net /SWITCH_5: track 16.0 -> 0.00 mm
- net +5V: track 201.0 -> 208.3 mm
- net Net-(F1-Pad2): track 4.93 -> 10.6 mm
- net /NET_C: track 14.6 -> 10.8 mm
Other:
- board text added: "SW6RL4 1.0 PDJR (c) 2021"
- board text removed: "THRMOD 1.0 PDJR (c) 2021"

Commit message: Updates
Parts:
- K1, K2, K3, K4: footprint PDJR:PCH-105L2MH -> PDJR:APAN-3105
- SW2: value PUSH_1 -> SW_MEC_5E; footprint Button_Switch_THT:SW_PUSH_6mm -> Button_Switch_THT:SW_PUSH_6mm_H4.3mm
- SW3: value PUSH_2 -> SW_MEC_5E; footprint Button_Switch_THT:SW_PUSH_6mm -> Button_Switch_THT:SW_PUSH_6mm_H4.3mm
- U1: value Teensy_3.2-PDJR -> Teensy_3.2
- U2: value TMR-1-1211 -> TMR-1211
- moved K2 9.65 mm to (188.9, 141.2)
- moved K3 6.86 mm to (160.7, 141.2)
- moved K1 4.06 mm to (194.7, 141.2)
- moved K4 1.27 mm to (154.9, 141.2)
Connections:
- SW2 pad 2: GND -> Net-(SW2-Pad2)
- SW3 pad 2: GND -> Net-(SW3-Pad2)
Routing:
- net +5V: track 208.3 -> 190.5 mm
- net Net-(K2-PadA1): track 30.9 -> 44.3 mm
- net Net-(J7-Pad1): track 6.71 -> 16.6 mm
- net Net-(J6-Pad2): track 16.4 -> 6.66 mm
- net Net-(J10-Pad2): track 16.4 -> 7.75 mm
- net Net-(J6-Pad1): track 6.71 -> 14.1 mm
- net Net-(K1-PadA1): track 44.6 -> 51.8 mm
- net Net-(J7-Pad2): track 16.4 -> 9.46 mm
- net Net-(J10-Pad1): track 6.71 -> 13.4 mm
- net /PUSH_2: track 117.8 -> 111.3 mm
- net /PUSH_1: track 130.7 -> 124.2 mm
- net Net-(J9-Pad1): track 6.71 -> 13.1 mm
- net Net-(K3-PadA1): track 18.7 -> 15.0 mm
- net Net-(J9-Pad2): track 16.4 -> 13.2 mm
- net Net-(K4-PadA1): track 6.44 -> 8.93 mm
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Other:
- board text removed: "PS+"
- board text removed: "PS-"
- board text removed: "PW+"
- board text removed: "PW-"
- board text removed: "RT+"
- board text removed: "RT-"
- board text removed: "SB+"
- board text removed: "SB-"
