File: TMP108/hardware/1.0/kicad/TMP108.kicad_pcb (KiCad board)
At the start: 2 copper layers, 75 x 75 mm, 38 parts, among them J1 Screw_Terminal_01x08, J2 Screw_Terminal_01x08, J3 CAN, SW1 PRG, SW2 SCR, SW3 PRG-VALUE, U1 Teensy_3.2, U2 TMR-1211, U3 MCP2551-I-P

Commit message: Updates
Routing:
- net /ADDR_0: track 5.61 -> 8.90 mm
- net /ADDR_1: track 8.95 -> 11.4 mm
- net /ADDR_2: track 11.7 -> 14.0 mm
- net /ADDR_6: track 26.0 -> 27.3 mm
- net /ADDR_5: track 22.5 -> 23.7 mm
- net /ADDR_3: track 15.3 -> 16.5 mm
- net /ADDR_4: track 18.9 -> 20.1 mm
- net /ADDR_7: track 29.7 -> 30.9 mm
- net GND: vias 0 -> 3
Other:
- board text added: "2022 (c) PDJR"
- board text added: "8"
- board text added: "THR108 1.1"
- board text removed: "2021 (c) PDJR"
- board text removed: "TSENSE 1.0"
